File: USB-CAN-Adapter.sch (EAGLE design)
At the start: 59 parts, among them IC1 STM32F303_F334_LQFP48, IC2 ISO1050DUB, IC3 FT232RL, IC4 78033, J8 CORTEX_DEBUGPTH, J9 USB-B, Y1 8MHz, Y2 32.768kHz

Commit message: board initial
Parts:
- removed C3: 100n, rcl:C-EUC0805
Connections:
- removed net CAN_GND: LED1.C
- removed net CAN_VCC: R2.2
- new net N$16: C18.2, J9.VBUS, L2.1
- net GND_CAN: now also LED1.C; no longer C3.2
- net LED_BLUE: now also IC1.PA3; no longer IC1.PB12
- net LED_RED: now also IC1.PA4; no longer IC1.PB13
- net VCC_CAN: now also R2.2; no longer C3.1
- net VCC_USB: no longer C18.2, J9.VBUS, L2.1
Changed lines of the file:
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@@
 <part name="IC1" library="STM32F303" deviceset="STM32F303_F334_LQFP48" device=""/>
 <part name="IC2" library="texas" deviceset="ISO1050" device="DUB"/>
-<part name="C3" library="rcl" deviceset="C-EU" device="C0805" value="100n"/>
 <part name="C4" library="rcl" deviceset="C-EU" device="C0805" value="100n"/>
 <part name="GND2" library="supply1" deviceset="GND" device=""/>
@@
 <instance part="IC1" gate="G$1" x="114.3" y="96.52"/>
 <instance part="IC2" gate="G$1" x="363.22" y="137.16" rot="R180"/>
-<instance part="C3" gate="G$1" x="444.5" y="76.2"/>
 <instance part="C4" gate="G$1" x="322.58" y="139.7"/>
 <instance part="GND2" gate="1" x="378.46" y="144.78" rot="R180"/>
@@
 </segment>
 <segment>
-<pinref part="IC1" gate="G$1" pin="VBAT"/>
-<wire x1="127" y1="144.78" x2="127" y2="160.02" width="0.1524" layer="91"/>
-<pinref part="P+6" gate="VCC" pin="VCC"/>
-</segment>
-<segment>
 <pinref part="R10" gate="G$1" pin="2"/>
 <wire x1="472.44" y1="-78.74" x2="472.44" y2="-76.2" width="0.1524" layer="91"/>
@@
 <pinref part="P+13" gate="VCC" pin="VCC"/>
 </segment>
+<segment>
+<pinref part="P+6" gate="VCC" pin="VCC"/>
+<pinref part="IC1" gate="G$1" pin="VBAT"/>
+<wire x1="127" y1="160.02" x2="127" y2="144.78" width="0.1524" layer="91"/>
+</segment>
 </net>
 <net name="CAN_L" class="0">
@@
 <wire x1="363.22" y1="-129.54" x2="355.6" y2="-129.54" width="0.1524" layer="91"/>
 <label x="363.22" y="-129.54" size="1.4224" layer="95" xref="yes"/>
-</segment>
-</net>
-<net name="CAN_VCC" class="0">
-<segment>
-<pinref part="R2" gate="G$1" pin="2"/>
-<wire x1="457.2" y1="-78.74" x2="457.2" y2="-76.2" width="0.1524" layer="91"/>
-<label x="457.2" y="-76.2" size="1.4224" layer="95" rot="R90" xref="yes"/>
-</segment>
-</net>
-<net name="CAN_GND" class="0">
-<segment>
-<pinref part="LED1" gate="G$1" pin="C"/>
-<wire x1="457.2" y1="-99.06" x2="457.2" y2="-101.6" width="0.1524" layer="91"/>
-<label x="457.2" y="-101.6" size="1.4224" layer="95" rot="R270" xref="yes"/>
 </segment>
 </net>
@@
 </segment>
 <segment>
-<pinref part="IC1" gate="G$1" pin="PB13"/>
-<wire x1="162.56" y1="104.14" x2="182.88" y2="104.14" width="0.1524" layer="91"/>
-<label x="182.88" y="104.14" size="1.4224" layer="95" xref="yes"/>
+<pinref part="IC1" gate="G$1" pin="PA4"/>
+<wire x1="66.04" y1="68.58" x2="55.88" y2="68.58" width="0.1524" layer="91"/>
+<label x="55.88" y="68.58" size="1.27" layer="95" rot="R180" xref="yes"/>
 </segment>
 </net>
@@
 </segment>
 <segment>
-<pinref part="IC1" gate="G$1" pin="PB12"/>
-<wire x1="162.56" y1="99.06" x2="182.88" y2="99.06" width="0.1524" layer="91"/>
-<label x="182.88" y="99.06" size="1.4224" layer="95" xref="yes"/>
+<pinref part="IC1" gate="G$1" pin="PA3"/>
+<wire x1="66.04" y1="73.66" x2="55.88" y2="73.66" width="0.1524" layer="91"/>
+<label x="55.88" y="73.66" size="1.27" layer="95" rot="R180" xref="yes"/>
 </segment>
 </net>
@@
 </net>
 <net name="VCC_USB" class="0">
-<segment>
-<pinref part="J9" gate="G$1" pin="VBUS"/>
-<wire x1="30.48" y1="-147.32" x2="40.64" y2="-147.32" width="0.1524" layer="91"/>
-<pinref part="C18" gate="G$1" pin="2"/>
-<wire x1="40.64" y1="-147.32" x2="40.64" y2="-142.24" width="0.1524" layer="91"/>
-<wire x1="40.64" y1="-147.32" x2="50.8" y2="-147.32" width="0.1524" layer="91"/>
-<junction x="40.64" y="-147.32"/>
-<wire x1="50.8" y1="-147.32" x2="50.8" y2="-114.3" width="0.1524" layer="91"/>
-<pinref part="L2" gate="G$1" pin="1"/>
-</segment>
 <segment>
 <pinref part="IC3" gate="1" pin="VCC"/>
@@
 <pinref part="DC1" gate="G$1" pin="+VOUT"/>
 <wire x1="411.48" y1="81.28" x2="429.26" y2="81.28" width="0.1524" layer="91"/>
-<pinref part="C3" gate="G$1" pin="1"/>
 <wire x1="429.26" y1="81.28" x2="444.5" y2="81.28" width="0.1524" layer="91"/>
 <wire x1="444.5" y1="81.28" x2="454.66" y2="81.28" width="0.1524" layer="91"/>
-<wire x1="444.5" y1="78.74" x2="444.5" y2="81.28" width="0.1524" layer="91"/>
 <pinref part="C2" gate="G$1" pin="1"/>
 <wire x1="429.26" y1="78.74" x2="429.26" y2="81.28" width="0.1524" layer="91"/>
@@
 <junction x="322.58" y="129.54"/>
 </segment>
+<segment>
+<pinref part="R2" gate="G$1" pin="2"/>
+<wire x1="457.2" y1="-78.74" x2="457.2" y2="-76.2" width="0.1524" layer="91"/>
+<label x="457.2" y="-76.2" size="1.4224" layer="95" rot="R90" xref="yes"/>
+</segment>
 </net>
 <net name="N$18" class="0">
@@
 <pinref part="C2" gate="G$1" pin="2"/>
 <wire x1="429.26" y1="68.58" x2="429.26" y2="71.12" width="0.1524" layer="91"/>
-<pinref part="C3" gate="G$1" pin="2"/>
 <wire x1="429.26" y1="68.58" x2="444.5" y2="68.58" width="0.1524" layer="91"/>
-<wire x1="444.5" y1="68.58" x2="444.5" y2="71.12" width="0.1524" layer="91"/>
 <wire x1="444.5" y1="68.58" x2="454.66" y2="68.58" width="0.1524" layer="91"/>
 <junction x="429.26" y="68.58"/>
@@
 <label x="363.22" y="-134.62" size="1.4224" layer="95" xref="yes"/>
 </segment>
-</net>
+<segment>
+<pinref part="LED1" gate="G$1" pin="C"/>
+<wire x1="457.2" y1="-99.06" x2="457.2" y2="-101.6" width="0.1524" layer="91"/>
+<label x="457.2" y="-101.6" size="1.4224" layer="95" rot="R270" xref="yes"/>
+</segment>
+</net>
+<net name="N$16" class="0">
+<segment>
+<pinref part="J9" gate="G$1" pin="VBUS"/>
+<pinref part="L2" gate="G$1" pin="1"/>
+<wire x1="30.48" y1="-147.32" x2="40.64" y2="-147.32" width="0.1524" layer="91"/>
+<wire x1="40.64" y1="-147.32" x2="50.8" y2="-147.32" width="0.1524" layer="91"/>
+<wire x1="50.8" y1="-147.32" x2="50.8" y2="-114.3" width="0.1524" layer="91"/>
+<pinref part="C18" gate="G$1" pin="2"/>
+<wire x1="40.64" y1="-142.24" x2="40.64" y2="-147.32" width="0.1524" layer="91"/>
+<junction x="40.64" y="-147.32"/>
+</segment>
+</net>
